File: capacitive-flex-sensor.kicad_pcb (KiCad board)
At the start: 2 copper layers, 331.5 x 48.5 mm, 13 parts, among them J3 Conn_01x12

Commit message: feat: new version with 5 pads and pins on top
Parts:
- removed CapPad10, CapPad11, CapPad12, CapPad6, CapPad7, CapPad8, CapPad9: ~, Sensor_Capacitive:capacitive_pad_35x17.5
- removed J3: Conn_01x12, Connector_PinHeader_2.54mm:PinHeader_1x12_P2.54mm_Vertical
- added J1: Conn_01x05, Connector_PinHeader_2.54mm:PinHeader_1x05_P2.54mm_Vertical, B.Cu at (124.1, 71.2)
- CapPad1, CapPad2, CapPad3, CapPad4, CapPad5: footprint Sensor_Capacitive:capacitive_pad_35x17.5 -> Sensor_Capacitive:capacitive_pad_20x20
- moved CapPad1 303.4 mm to (160.6, 105.4)
- moved CapPad2 294.6 mm to (134.5, 105.3)
- moved CapPad3 286.0 mm to (108.5, 105.4)
- moved CapPad4 277.8 mm to (82.5, 105.4)
- moved CapPad5 270.0 mm to (56.5, 105.3)
Routing:
- net Net-(J3-Pin_6): track 307.8 -> 0.00 mm, vias 2 -> 0
- net Net-(J3-Pin_12): track 303.4 -> 0.00 mm, vias 2 -> 0
- net Net-(J3-Pin_11): track 264.1 -> 0.00 mm, vias 2 -> 0
- net Net-(J3-Pin_10): track 226.6 -> 0.00 mm, vias 2 -> 0
- net Net-(J1-Pin_5): track 265.6 -> 61.7 mm, vias 2 -> 0
- net Net-(J3-Pin_9): track 188.5 -> 0.00 mm, vias 2 -> 0
- net Net-(J1-Pin_4): track 221.0 -> 39.4 mm, vias 2 -> 0
- net Net-(J1-Pin_3): track 182.0 -> 24.4 mm, vias 2 -> 0
- net Net-(J3-Pin_8): track 150.2 -> 0.00 mm, vias 2 -> 0
- net Net-(J3-Pin_7): track 106.8 -> 0.00 mm
- net Net-(J1-Pin_2): track 143.4 -> 38.3 mm, vias 2 -> 0
- net Net-(J1-Pin_1): track 106.5 -> 60.8 mm
Other:
- board size 331.5 x 48.5 mm -> 160.7 x 48.1 mm
- board text added: "Designed by: Jehan Yang Version: 1.0 - 03/2024"

Commit message: chore: change version number on layout
Parts:
- J1: moved to F.Cu
- moved J1 0.08 mm to (124.1, 71.2), turned to -90 degrees
Other:
- board text added: "Designed by: Jehan Yang Version: 1.1 - 03/2024"
- board text removed: "Designed by: Jehan Yang Version: 1.0 - 03/2024"
Changed lines of the file:
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@@
       (net 4 "Net-(J1-Pin_4)") (pinfunction "1") (pintype "output"))
+  )
+  (footprint "Connector_PinHeader_2.54mm:PinHeader_1x05_P2.54mm_Vertical" (layer "F.Cu")
+    (at 124.14 71.16 -90)
+    (descr "Through hole straight pin header, 1x05, 2.54mm pitch, single row")
+    (tags "Through hole pin header THT 1x05 2.54mm single row")
+    (property "Sheetfile" "capacitive-flex-sensor.kicad_sch")
+    (property "Sheetname" "")
+    (property "ki_description" "Generic connector, single row, 01x05, script generated (kicad-library-utils/schlib/autogen/connector/)")
+    (property "ki_keywords" "connector")
+    (attr through_hole)
+    (fp_text reference "J1" (at -2.7 5.03 -180) (layer "F.SilkS")
+        (effects (font (size 1 1) (thickness 0.15)))
+    )
+    (fp_text value "Conn_01x05" (at -3.6 4.85) (layer "F.Fab")
+        (effects (font (size 1 1) (thickness 0.15)))
+    )
+    (fp_text user "${REFERENCE}" (at 0 5.08) (layer "F.Fab")
+        (effects (font (size 1 1) (thickness 0.15)))
+    )
+    (fp_line (start -1.33 -1.33) (end 0 -1.33)
+      (stroke (width 0.12) (type solid)) (layer "F.SilkS"))
+    (fp_line (start -1.33 0) (end -1.33 -1.33)
+      (stroke (width 0.12) (type solid)) (layer "F.SilkS"))
+    (fp_line (start -1.33 1.27) (end -1.33 11.49)
+      (stroke (width 0.12) (type solid)) (layer "F.SilkS"))
+    (fp_line (start -1.33 1.27) (end 1.33 1.27)
+      (stroke (width 0.12) (type solid)) (layer "F.SilkS"))
+    (fp_line (start -1.33 11.49) (end 1.33 11.49)
+      (stroke (width 0.12) (type solid)) (layer "F.SilkS"))
+    (fp_line (start 1.33 1.27) (end 1.33 11.49)
+      (stroke (width 0.12) (type solid)) (layer "F.SilkS"))
+    (fp_line (start -1.8 -1.8) (end -1.8 11.95)
+      (stroke (width 0.05) (type solid)) (layer "F.CrtYd"))
+    (fp_line (start -1.8 11.95) (end 1.8 11.95)
+      (stroke (width 0.05) (type solid)) (layer "F.CrtYd"))
+    (fp_line (start 1.8 -1.8) (end -1.8 -1.8)
+      (stroke (width 0.05) (type solid)) (layer "F.CrtYd"))
+    (fp_line (start 1.8 11.95) (end 1.8 -1.8)
+      (stroke (width 0.05) (type solid)) (layer "F.CrtYd"))
+    (fp_line (start -1.27 -0.635) (end -0.635 -1.27)
+      (stroke (width 0.1) (type solid)) (layer "F.Fab"))
+    (fp_line (start -1.27 11.43) (end -1.27 -0.635)
+      (stroke (width 0.1) (type solid)) (layer "F.Fab"))
+    (fp_line (start -0.635 -1.27) (end 1.27 -1.27)
+      (stroke (width 0.1) (type solid)) (layer "F.Fab"))
+    (fp_line (start 1.27 -1.27) (end 1.27 11.43)
+      (stroke (width 0.1) (type solid)) (layer "F.Fab"))
+    (fp_line (start 1.27 11.43) (end -1.27 11.43)
+      (stroke (width 0.1) (type solid)) (layer "F.Fab"))
+    (pad "1" thru_hole rect (at 0 0 270) (size 1.7 1.7) (drill 1) (layers "*.Cu" "*.Mask")
+      (net 1 "Net-(J1-Pin_1)") (pinfunction "Pin_1") (pintype "passive"))
+    (pad "2" thru_hole oval (at 0 2.54 270) (size 1.7 1.7) (drill 1) (layers "*.Cu" "*.Mask")
+      (net 2 "Net-(J1-Pin_2)") (pinfunction "Pin_2") (pintype "passive"))
+    (pad "3" thru_hole oval (at 0 5.08 270) (size 1.7 1.7) (drill 1) (layers "*.Cu" "*.Mask")
+      (net 3 "Net-(J1-Pin_3)") (pinfunction "Pin_3") (pintype "passive"))
+    (pad "4" thru_hole oval (at 0 7.62 270) (size 1.7 1.7) (drill 1) (layers "*.Cu" "*.Mask")
+      (net 4 "Net-(J1-Pin_4)") (pinfunction "Pin_4") (pintype "passive"))
+    (pad "5" thru_hole oval (at 0 10.16 270) (size 1.7 1.7) (drill 1) (layers "*.Cu" "*.Mask")
+      (net 5 "Net-(J1-Pin_5)") (pinfunction "Pin_5") (pintype "passive"))
+    (model "${KICAD6_3DMODEL_DIR}/Connector_PinHeader_2.54mm.3dshapes/PinHeader_1x05_P2.54mm_Vertical.wrl"
+      (offset (xyz 0 0 0))
+      (scale (xyz 1 1 1))
+      (rotate (xyz 0 0 0))
+    )
   )
   (footprint "Sensor_Capacitive:capacitive_pad_20x20" (layer "F.Cu")
@@
       (net 1 "Net-(J1-Pin_1)") (pinfunction "1") (pintype "output"))
   )
-  (footprint "Connector_PinHeader_2.54mm:PinHeader_1x05_P2.54mm_Vertical" (layer "B.Cu")
-    (at 124.135 71.24 90)
-    (descr "Through hole straight pin header, 1x05, 2.54mm pitch, single row")
-    (tags "Through hole pin header THT 1x05 2.54mm single row")
-    (property "Sheetfile" "capacitive-flex-sensor.kicad_sch")
-    (property "Sheetname" "")
-    (property "ki_description" "Generic connector, single row, 01x05, script generated (kicad-library-utils/schlib/autogen/connector/)")
-    (property "ki_keywords" "connector")
-    (attr through_hole)
-    (fp_text reference "J1" (at 2.39 -5.26) (layer "F.SilkS")
-        (effects (font (size 1 1) (thickness 0.15)))
-    )
-    (fp_text value "Conn_01x05" (at -3.6 -4.85) (layer "B.Fab")
-        (effects (font (size 1 1) (thickness 0.15)) (justify mirror))
-    )
-    (fp_text user "${REFERENCE}" (at 0 -5.08) (layer "B.Fab")
-        (effects (font (size 1 1) (thickness 0.15)) (justify mirror))
-    )
-    (fp_line (start -1.33 -11.49) (end 1.33 -11.49)
-      (stroke (width 0.12) (type solid)) (layer "B.SilkS"))
-    (fp_line (start -1.33 -1.27) (end -1.33 -11.49)
-      (stroke (width 0.12) (type solid)) (layer "B.SilkS"))
-    (fp_line (start -1.33 -1.27) (end 1.33 -1.27)
-      (stroke (width 0.12) (type solid)) (layer "B.SilkS"))
-    (fp_line (start -1.33 0) (end -1.33 1.33)
-      (stroke (width 0.12) (type solid)) (layer "B.SilkS"))
-    (fp_line (start -1.33 1.33) (end 0 1.33)
-      (stroke (width 0.12) (type solid)) (layer "B.SilkS"))
-    (fp_line (start 1.33 -1.27) (end 1.33 -11.49)
-      (stroke (width 0.12) (type solid)) (layer "B.SilkS"))
-    (fp_line (start -1.8 -11.95) (end 1.8 -11.95)
-      (stroke (width 0.05) (type solid)) (layer "B.CrtYd"))
-    (fp_line (start -1.8 1.8) (end -1.8 -11.95)
-      (stroke (width 0.05) (type solid)) (layer "B.CrtYd"))
-    (fp_line (start 1.8 -11.95) (end 1.8 1.8)
-      (stroke (width 0.05) (type solid)) (layer "B.CrtYd"))
-    (fp_line (start 1.8 1.8) (end -1.8 1.8)
-      (stroke (width 0.05) (type solid)) (layer "B.CrtYd"))
-    (fp_line (start -1.27 -11.43) (end -1.27 0.635)
-      (stroke (width 0.1) (type solid)) (layer "B.Fab"))
-    (fp_line (start -1.27 0.635) (end -0.635 1.27)
-      (stroke (width 0.1) (type solid)) (layer "B.Fab"))
-    (fp_line (start -0.635 1.27) (end 1.27 1.27)
-      (stroke (width 0.1) (type solid)) (layer "B.Fab"))
-    (fp_line (start 1.27 -11.43) (end -1.27 -11.43)
-      (stroke (width 0.1) (type solid)) (layer "B.Fab"))
-    (fp_line (start 1.27 1.27) (end 1.27 -11.43)
-      (stroke (width 0.1) (type solid)) (layer "B.Fab"))
-    (pad "1" thru_hole rect (at 0 0 90) (size 1.7 1.7) (drill 1) (layers "*.Cu" "*.Mask")
-      (net 1 "Net-(J1-Pin_1)") (pinfunction "Pin_1") (pintype "passive"))
-    (pad "2" thru_hole oval (at 0 -2.54 90) (size 1.7 1.7) (drill 1) (layers "*.Cu" "*.Mask")
-      (net 2 "Net-(J1-Pin_2)") (pinfunction "Pin_2") (pintype "passive"))
-    (pad "3" thru_hole oval (at 0 -5.08 90) (size 1.7 1.7) (drill 1) (layers "*.Cu" "*.Mask")
-      (net 3 "Net-(J1-Pin_3)") (pinfunction "Pin_3") (pintype "passive"))
-    (pad "4" thru_hole oval (at 0 -7.62 90) (size 1.7 1.7) (drill 1) (layers "*.Cu" "*.Mask")
-      (net 4 "Net-(J1-Pin_4)") (pinfunction "Pin_4") (pintype "passive"))
-    (pad "5" thru_hole oval (at 0 -10.16 90) (size 1.7 1.7) (drill 1) (layers "*.Cu" "*.Mask")
-      (net 5 "Net-(J1-Pin_5)") (pinfunction "Pin_5") (pintype "passive"))
-    (model "${KICAD6_3DMODEL_DIR}/Connector_PinHeader_2.54mm.3dshapes/PinHeader_1x05_P2.54mm_Vertical.wrl"
-      (offset (xyz 0 0 0))
-      (scale (xyz 1 1 1))
-      (rotate (xyz 0 0 0))
-    )
-  )
   (gr_rect (start 299.375 88.26) (end 305.985 124.72)
     (stroke (width 0.1) (type default)) (fill none) (layer "Dwgs.User"))
@@
   (gr_line (start 129.13 115.41) (end 40.81925 115.41)
     (stroke (width 0.1) (type default)) (layer "Edge.Cuts"))
-  (gr_text "Designed by: Jehan Yang\nVersion: 1.0 - 03/2024\n" (at 183.85 113.35) (layer "B.SilkS")
+  (gr_text "Designed by: Jehan Yang\nVersion: 1.1 - 03/2024\n" (at 183.85 113.35) (layer "B.SilkS")
     (effects (font (size 1 1) (thickness 0.15)) (justify left bottom mirror))
   )
